File: PCB/Sensor/Argos_Battery_Charge_Monitor_Sensor.brd (EAGLE design)
At the start: 160 x 100 mm, 24 parts, among them J1 AVR_SPI_PRG_62X3_LOCK, U1 L78M05CDT-TR

Commit message: 2017 RevA boards complete
Parts:
- added C1, C2, C3: 0.1uF, SparkFun-Capacitors:0805
- moved V_CHARGE_IN 93.3 mm to (44.5, 21.1)
- moved R3 92.8 mm to (40.6, 19.1), turned to 90 degrees
- moved R9 87.8 mm to (24.1, 2.54), flipped to the bottom
- moved R8 87.4 mm to (40.6, 2.54), flipped to the bottom, turned to 180 degrees
- moved R10 83.2 mm to (19.1, 2.54), flipped to the bottom
- moved U$2 82.3 mm to (39.4, 17.3), flipped to the bottom, turned to 270 degrees
- moved R2 81.6 mm to (31.8, 16.5), turned to 180 degrees
- moved GND_OUT 80.9 mm to (50.8, 13.5)
- moved R7 80.3 mm to (35.6, 2.54), flipped to the bottom, turned to 180 degrees
- moved V_CHARGE_OUT 79.8 mm to (44.5, 13.5)
- moved R11 79.0 mm to (14.0, 2.54), flipped to the bottom
- moved R1 77.1 mm to (31.8, 19.1), turned to 180 degrees
- moved R6 73.7 mm to (30.5, 2.54), flipped to the bottom, turned to 180 degrees
- moved GND_IN 72.1 mm to (50.8, 21.1)
- moved U$3 71.7 mm to (26.7, 12.7), flipped to the bottom, turned to 270 degrees
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Connections:
- net 5V: now also C1.1, C2.1, C3.1
- net GND: now also C1.2, C2.2, C3.2
- net N$2: now also U$6.6; no longer U$6.5
- net N$3: now also U$6.7; no longer U$6.6
- net N$4: now also U$6.8; no longer U$6.7
- net N$5: now also U$6.5; no longer U$6.8
Routing:
- net D_SDA_M: track 0.00 -> 33.7 mm, vias 0 -> 1
- net D_SCK_M: track 0.00 -> 31.2 mm, vias 0 -> 1
- net SCL: track 0.00 -> 31.2 mm, vias 0 -> 1
- net SDA: track 0.00 -> 30.0 mm, vias 0 -> 1
- net D_SDA_P: track 0.00 -> 29.6 mm, vias 0 -> 1
- net D_SCK_P: track 0.00 -> 29.2 mm, vias 0 -> 1
- net N$1: track 0.00 -> 27.5 mm, vias 0 -> 1
- net N$8: track 0.00 -> 22.7 mm, vias 0 -> 2
- net N$6: track 0.00 -> 20.8 mm, vias 0 -> 1
- net N$11: track 0.00 -> 18.6 mm, vias 0 -> 1
- net N$15: track 0.00 -> 16.2 mm, vias 0 -> 1
- net 5V: track 0.00 -> 15.2 mm, vias 0 -> 3
- net N$16: track 0.00 -> 13.7 mm
- net N$13: track 0.00 -> 13.2 mm
- net N$5: track 0.00 -> 9.45 mm
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- added copper zone on layer 1, net 5V
- added copper zone on layer 16, net GND
- added copper zone on layer 16, net N$7
- added copper zone on layer 16, net N$9
Other:
- board size 160 x 100 mm -> 58.4 x 32.7 mm
- board text added: "+"
- board text added: "-"
- board text added: "1"
- board text added: "2"
- board text added: "4"
- board text added: "5V"
- board text added: "8"
- board text added: "Argos Battery Charge Monitor Sensor Rev 2017A github.com/FRC1756-Argos"
- board text added: "C1"
- board text added: "CHARGER IN"
- board text added: "CHARGER OUT"
- board text added: "GND"
- board text added: "I2C Addr"
- board text added: "ICSP"
- board text added: "MISO"
- board text added: "MOSI"
- board text added: "R1"
- board text added: "R2"
- board text added: "R3"
- board text added: "R4"
- board text added: "R5"
- board text added: "R6"
- board text added: "RST"
- board text added: "SCK"
- board text added: "SCL TERM"
- board text added: "SDA TERM"
- board text added: "STATUS"
- board text added: "U1"
- board text added: "U2"
- board text added: "U3"
- board text added: "U4"
