File: PCB/Sensor/Argos_Battery_Charge_Monitor_Sensor.sch (EAGLE design)
At the start: 24 parts, among them J1 AVR_SPI_PRG_62X3_LOCK, U1 L78M05CDT-TR

Commit message: 2017 RevA boards complete
Parts:
- added C1, C2, C3: 0.1uF, SparkFun-Capacitors:CAP0805
Connections:
- net 5V: now also C1.1, C2.1, C3.1
- net GND: now also C1.2, C2.2, C3.2
- net N$2: now also U$6.6; no longer U$6.5
- net N$3: now also U$6.7; no longer U$6.6
- net N$4: now also U$6.8; no longer U$6.7
- net N$5: now also U$6.5; no longer U$6.8
